Commit message: Add IMU sensor to URDF and launch, add imu_subscriber node
- Add IMU link, joint, and sensor to robot.urdf - Update launch file to
bridge IMU topic from Gazebo - Add imu_subscriber.py node to subscribe
and log IMU data - Install imu_subscriber.py in CMakeLists.txt

File: wheelchair_ros/wheelchair/robot.urdf (robot description, URDF)
Before this commit: robot nishcorp_wheelchair, 11 links, 10 joints
Links:
- added link imu_link, mass 0.01; collision box size=0.02 0.02 0.02; visual box size=0.02 0.02 0.02
Joints:
- added joint imu_joint: type fixed, parent fiberglass_seat_v3_v9, child imu_link, origin xyz=0 0 0.1 rpy=0 0 0
